File: Main board.kicad_pcb (KiCad board)
At the start: 4 copper layers, 50 x 75 mm, 101 parts, among them CN1 KF127S-3.5-6P, CN2 KF127S-3.5-6P, J1 Conn_ARM_SWD_TagConnect_TC203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, J2 Conn_01x02_Pin, J3 Micro-Fit 43650-0215, J5 Connector, USB-TYPE-C-16P, J6 Micro-Fit 43650-0215, J7 Conn_01x02_Pin, J8 Conn_01x04_Pin, Q1 SI7232DN-T1-GE3, Q2 SI7232DN-T1-GE3, SW1 SKRKAEE020, SW2 SKRKAEE020, U1 STM32U575VGTx, U10 TLV75733PDBV, U11 NRVB120VLSFT1G, U12 NRVB120VLSFT1G, U2 TPS62901RPJR, U3 MS5607-02BA03, U9 ICM-45686, X1 1XXD32000MBA, Y1 ECS-327TXO-33-TR

Commit message: +Ejection area
-almost finish routing ejection part
-5V buck copied from Tata
- Moves and update.ioc file for better route
-USB C needs some rework?
Parts:
- moved H3 82.6 mm to (168.4, 109.5)
- moved J7 76.2 mm to (168.4, 89.0), turned to -90 degrees
- moved R22 65.5 mm to (161.3, 77.9), turned to 180 degrees
- moved J5 64.4 mm to (166.0, 76.6)
- moved R23 64.4 mm to (161.1, 75.0)
- moved D1 58.5 mm to (160.6, 83.8)
- moved C26 54.3 mm to (160.1, 86.4)
- moved C28 54.0 mm to (155.1, 97.0), turned to 180 degrees
- moved U11 52.5 mm to (158.9, 88.5)
- moved C27 52.5 mm to (151.7, 98.8), turned to 90 degrees
- moved J8 51.3 mm to (123.2, 85.5), turned to 180 degrees
- moved U10 50.4 mm to (153.8, 90.0)
- moved C35 50.4 mm to (150.9, 90.1)
- moved C36 50.4 mm to (157.9, 90.3)
- moved L1 49.5 mm to (160.9, 98.2), turned to -90 degrees
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Connections:
- J8 pad 2: USART3_RX -> USART4_RX
- J8 pad 3: USART3_TX -> USART4_TX
- R40 pad 1: PYRO+ -> Net-(JP3-C)
- R42 pad 1: PYRO+ -> Net-(JP4-C)
- U1 pad 23: unconnected-(U1-PA0-Pad23) -> USART4_TX
- U1 pad 24: unconnected-(U1-PA1-Pad24) -> USART4_RX
- U1 pad 25: FIRE_B -> unconnected-(U1-PA2-Pad25)
- U1 pad 26: FIRE_A -> unconnected-(U1-PA3-Pad26)
- U1 pad 33: USART3_TX -> unconnected-(U1-PC4-Pad33)
- U1 pad 34: USART3_RX -> unconnected-(U1-PC5-Pad34)
- U1 pad 40: SERVO1 -> unconnected-(U1-PE9-Pad40)
- U1 pad 42: SERVO2 -> FIRE_A
- U1 pad 43: unconnected-(U1-PE12-Pad43) -> FIRE_B
- U1 pad 44: unconnected-(U1-PE13-Pad44) -> SERVO1
- U1 pad 45: unconnected-(U1-PE14-Pad45) -> SERVO2
- U1 pad 46: unconnected-(U1-PE15-Pad46) -> FIRE_D
- U1 pad 47: unconnected-(U1-PB10-Pad47) -> FIRE_C
- U1 pad 53: DAT0 -> unconnected-(U1-PB14-Pad53)
- U1 pad 54: DAT1 -> unconnected-(U1-PB15-Pad54)
- U1 pad 65: unconnected-(U1-PC8-Pad65) -> DAT0
- U1 pad 66: unconnected-(U1-PC9-Pad66) -> DAT1
- U1 pad 67: MS5607_CS -> unconnected-(U1-PA8-Pad67)
- U1 pad 7: FIRE_C -> unconnected-(U1-PC13-Pad7)
- U1 pad 78: unconnected-(U1-PC10-Pad78) -> DAT2
- U1 pad 79: unconnected-(U1-PC11-Pad79) -> DAT3
- U1 pad 80: unconnected-(U1-PC12-Pad80) -> SDMMC_CLK
- U1 pad 81: unconnected-(U1-PD0-Pad81) -> MS5607_CS
- U1 pad 83: unconnected-(U1-PD2-Pad83) -> SDMMC_CMD
- U1 pad 87: SDMMC_CLK -> unconnected-(U1-PD6-Pad87)
- U1 pad 88: SDMMC_CMD -> unconnected-(U1-PD7-Pad88)
- U1 pad 89: DAT2 -> unconnected-(U1-PB3-Pad89)
- U1 pad 9: FIRE_D -> unconnected-(U1-PC15-Pad9)
- U1 pad 90: DAT3 -> unconnected-(U1-PB4-Pad90)
Routing:
- net SERVO2: track 0.00 -> 53.5 mm, vias 0 -> 1
- net SERVO1: track 0.00 -> 39.0 mm, vias 0 -> 1
- net BEC+: track 0.00 -> 38.4 mm, vias 0 -> 12
- net Net-(JP3-C): track 0.00 -> 25.8 mm, vias 0 -> 7
- net Net-(JP4-C): track 0.00 -> 25.7 mm, vias 0 -> 7
- net USART1_RX: track 0.00 -> 23.4 mm, vias 0 -> 1
- net USART1_TX: track 0.00 -> 22.2 mm, vias 0 -> 1
- net FIRE_A: track 0.00 -> 17.9 mm
- net FIRE_B: track 0.00 -> 17.2 mm
- net D-: track 0.00 -> 13.3 mm
- net D+: track 0.00 -> 11.9 mm, vias 0 -> 3
- net Net-(Q1-G2): track 0.00 -> 11.5 mm, vias 0 -> 2
- net Net-(Q1-G1): track 0.00 -> 9.84 mm, vias 0 -> 2
- net VBAT+: track 6.13 -> 0.44 mm, vias 0 -> 9
- net VBUS: track 0.00 -> 5.66 mm
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- added copper zone on F.Cu, net +5V
- added copper zone on In2.Cu, net +5V
- added copper zone on F.Cu, net BEC+
- added copper zone on In2.Cu, net BEC+
- added copper zone on F.Cu, net Net-(CN2-Pad6)
- added copper zone on F.Cu, net Net-(U2-SW)
- added copper zone on F.Cu, net PYRO_GND
- added copper zone on In2.Cu, net VBAT+
- added copper zone on In1.Cu, net VBAT-
Other:
- board text added: "CKCS4018-1UH/N"
- board text added: "REF**"

Commit message: Some layout changes by Tata
Parts:
- moved C36 93.7 mm to (251.2, 98.5)
- moved U10 93.7 mm to (247.1, 98.2)
- moved U11 93.7 mm to (252.3, 96.8)
- moved U12 93.7 mm to (250.4, 101.6)
- moved C35 93.7 mm to (244.2, 98.3)
- moved C27 49.7 mm to (196.1, 120.9)
- moved C28 49.7 mm to (199.5, 119.1)
- moved C29 49.7 mm to (199.1, 126.0)
- moved L1 49.7 mm to (205.4, 120.3)
- moved R24 49.7 mm to (201.8, 125.9)
- moved R25 49.7 mm to (195.9, 124.1)
- moved R26 49.7 mm to (205.1, 125.1)
- moved U2 49.7 mm to (199.9, 122.1)
- moved JP1 42.6 mm to (151.9, 146.9)
- moved C31 42.6 mm to (170.5, 146.0)
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Routing:
- net SERVO2: track 53.5 -> 0.00 mm, vias 1 -> 0
- net SERVO1: track 39.0 -> 0.00 mm, vias 1 -> 0
- net BEC+: track 38.4 -> 0.00 mm, vias 12 -> 0
- net Net-(JP3-C): track 25.8 -> 0.00 mm, vias 7 -> 0
- net Net-(JP4-C): track 25.7 -> 0.00 mm, vias 7 -> 0
- net USART1_RX: track 23.4 -> 0.00 mm, vias 1 -> 0
- net USART1_TX: track 22.2 -> 0.00 mm, vias 1 -> 0
- net FIRE_A: track 17.9 -> 0.00 mm
- net FIRE_B: track 17.2 -> 0.00 mm
- net D-: track 13.3 -> 0.00 mm
- net D+: track 11.9 -> 0.00 mm, vias 3 -> 0
- net Net-(Q1-G2): track 11.5 -> 0.00 mm, vias 2 -> 0
- net Net-(Q1-G1): track 9.84 -> 0.00 mm, vias 2 -> 0
- net VBUS: track 5.66 -> 0.00 mm
- net Net-(CN1-Pad1): track 4.74 -> 0.00 mm
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- removed copper zone on In2.Cu, net +5V
- removed copper zone on F.Cu, net BEC+
- removed copper zone on In2.Cu, net BEC+
- removed copper zone on F.Cu, net Net-(CN1-Pad1)
- removed copper zone on F.Cu, net Net-(CN1-Pad2)
- removed copper zone on F.Cu, net Net-(CN2-Pad5)
- removed copper zone on F.Cu, net Net-(CN2-Pad6)
- removed copper zone on F.Cu, net Net-(U10-EN)
- removed copper zone on In2.Cu, net VBAT+
