File: Main board.kicad_sch (KiCad schematic)
At the start: 103 parts, among them CN1 KF127S-3.5-6P, CN2 KF127S-3.5-6P, J1 Conn_ARM_SWD_TagConnect_TC203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, J2 Conn_01x02_Pin, J3 Micro-Fit 43650-0215, J5 Connector, USB-TYPE-C-16P, J6 Micro-Fit 43650-0215, J7 Conn_01x02_Pin, J8 Conn_01x04_Pin, Q1 SI7232DN-T1-GE3, Q2 SI7232DN-T1-GE3, SW1 SKRKAEE020, SW2 SKRKAEE020, U1 STM32U575VGTx, U10 TLV75733PDBV, U11 NRVB120VLSFT1G, U12 NRVB120VLSFT1G, U2 TPS62901RPJR, U7 SN74AHCT125DR, X1 1XXD32000MBA, Y1 ECS-327TXO-33-TR

Commit message: +Ejection area
-almost finish routing ejection part
-5V buck copied from Tata
- Moves and update.ioc file for better route
-USB C needs some rework?
Connections:
- net DAT0: now also U1.65 (PC8); no longer U1.53 (PB14)
- net DAT1: now also U1.66 (PC9); no longer U1.54 (PB15)
- net DAT2: now also U1.78 (PC10); no longer U1.89 (PB3)
- net DAT3: now also U1.79 (PC11); no longer U1.90 (PB4)
- net FIRE_A: now also U1.42 (PE11); no longer U1.26 (PA3)
- net FIRE_B: now also U1.43 (PE12); no longer U1.25 (PA2)
- net FIRE_C: now also U1.47 (PB10); no longer U1.7 (PC13)
- net FIRE_D: now also U1.46 (PE15); no longer U1.9 (PC15)
- net MS5607_CS: now also U1.81 (PD0); no longer U1.67 (PA8)
- net PYRO+: no longer R40.1, R42.1
- net SDMMC_CLK: now also U1.80 (PC12); no longer U1.87 (PD6)
- net SDMMC_CMD: now also U1.83 (PD2); no longer U1.88 (PD7)
- net SERVO1: now also U1.44 (PE13); no longer U1.40 (PE9)
- net SERVO2: now also U1.45 (PE14); no longer U1.42 (PE11)
- net at CN2.2, JP4.2 (C): now also R42.1
- net at CN1.5, JP3.2 (C): now also R40.1
- net USART4_TX: now reaches U1.23 (PA0)
- net USART4_TX: now also J8.3 (Pin_3)
- net USART4_RX: now reaches U1.24 (PA1)
- net USART4_RX: now also J8.2 (Pin_2)
- net USART3_RX: no longer names the net of U1.34 (PC5)
- net USART3_RX: no longer J8.2 (Pin_2)
- net USART3_TX: no longer names the net of U1.33 (PC4)
- net USART3_TX: no longer J8.3 (Pin_3)
Other:
- moved on the sheet: R15, R40, R42

Commit message: Some layout changes by Tata
Other:
- note added: "Output TO BEC"
Changed lines of the file:
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@@
+		)
+	)
+	(text "Output TO BEC"
+		(exclude_from_sim no)
+		(at 99.06 100.33 0)
+		(effects
+			(font
+				(size 1.27 1.27)
+			)
 		)
 	)
